Commit message: Finalised universal robot filed for ROAR arm

File: Assembly_description/urdf/panda_example.urdf (robot description, URDF)
Before this commit: robot panda, 9 links, 8 joints
Links:
- link panda_link0: mass 2.8142028896 -> None; geometry collision mesh filename=package://franka_description/meshes/collision/link0.stl; visual mesh filename=package://franka_description/meshes/collision/link0.stl
- link panda_link1: mass 2.3599995791 -> None; geometry collision mesh filename=package://franka_description/meshes/collision/link1.stl; visual mesh filename=package://franka_description/meshes/collision/link1.stl
- link panda_link2: mass 2.379518833 -> None; geometry collision mesh filename=package://franka_description/meshes/collision/link2.stl; visual mesh filename=package://franka_description/meshes/collision/link2.stl
- link panda_link3: mass 2.6498823337 -> None; geometry collision mesh filename=package://franka_description/meshes/collision/link3.stl; visual mesh filename=package://franka_description/meshes/collision/link3.stl
- link panda_link4: mass 2.6948018744 -> None; geometry collision mesh filename=package://franka_description/meshes/collision/link4.stl; visual mesh filename=package://franka_description/meshes/collision/link4.stl
- link panda_link5: mass 2.9812816864 -> None; geometry collision mesh filename=package://franka_description/meshes/collision/link5.stl; visual mesh filename=package://franka_description/meshes/collision/link5.stl
- link panda_link6: mass 1.1285806309 -> None; geometry collision mesh filename=package://franka_description/meshes/collision/link6.stl; visual mesh filename=package://franka_description/meshes/collision/link6.stl
- link panda_link7: mass 0.4052912465 -> None; geometry collision mesh filename=package://franka_description/meshes/collision/link7.stl; visual mesh filename=package://franka_description/meshes/collision/link7.stl
